File: Arduino_MEGA_2560-Rev3_Shield.brd (EAGLE design)
At the start: 93.4 x 53.3 mm, 44 parts, among them IC1 785.0RECOM

Commit message: Synching real boards with git repo
Parts:
- C1: value (none) -> 10uF
- moved SR04-5 11.4 mm to (63.5, 40.6)
- moved SR04-6 11.4 mm to (63.5, 35.6)
- moved SR04-7 11.4 mm to (63.5, 17.8)
- moved SR04-8 11.4 mm to (63.5, 12.7)
- moved XIO 11.4 mm to (83.8, 29.2)
- moved ADCL 11.4 mm to (48.3, 2.54)
- moved ADCL1 11.4 mm to (48.3, 5.08)
- moved C1 11.4 mm to (22.6, 26.7)
- moved I2C 11.4 mm to (7.62, 7.62)
- moved IC1 11.4 mm to (9.40, 21.6)
- moved IR1 11.4 mm to (47.0, 40.6)
- moved IR2 11.4 mm to (47.0, 35.6)
- moved IR3 11.4 mm to (47.0, 17.8)
- moved IR4 11.4 mm to (47.0, 12.7)
- moved JP1 11.4 mm to (18.8, 48.3)
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Connections:
- net N$1 renamed PB7
- net N$10 renamed SDA&2
- net N$11 renamed SCL&2
- net N$13 renamed PG5
- net N$16 renamed TX0
- net N$17 renamed RX0
- net N$19 renamed ADC7
- net N$20 renamed ADC6
- net N$21 renamed ADC5
- net N$22 renamed ADC4
- net N$23 renamed ADC3
- net N$24 renamed ADC2
- net N$25 renamed ADC1
- net N$26 renamed ADC0
- net N$3 renamed PB6
- net N$4 renamed PB5
- net N$5 renamed PB4
- net N$8 renamed TXD1
- net N$9 renamed RXD1
- removed net N$6: JP1.9, JP6.9
- removed net PD7: XIO.19
- new net PC6: XIO.12
- new net PE3: PWML.6, PWML1.6
- net IR1: now also XIO.3; no longer XIO.18
- net IR2: now also XIO.4; no longer XIO.17
- net IR3: now also XIO.19; no longer XIO.16
- net IR4: now also XIO.28; no longer XIO.15
- net IR5: now also XIO.9; no longer XIO.14
- net IR6: now also XIO.10; no longer XIO.13
- net IR7: now also XIO.29; no longer XIO.12
- net IR8: now also XIO.30; no longer XIO.11
- net L1: now also PWML.8, PWML1.8; no longer PWML.6, PWML1.6
- net L2: now also PWML.7, PWML1.7; no longer PWML.3, PWML1.3
- net L3: now also JP1.10, JP6.10; no longer PWML.4, PWML1.4
- net L4: now also JP1.9, JP6.9; no longer PWML.7, PWML1.7
- net L5: now also XIO.27; no longer PWML.8, PWML1.8
- net L6: now also XIO.26; no longer JP1.10, JP6.10
- net L7: now also XIO.25; no longer XIO.27
- net L8: now also PWML.3, PWML1.3; no longer XIO.26
- net L9: now also PWML.4, PWML1.4; no longer XIO.25
- net U1-E: now also XIO.13; no longer XIO.3
- net U1-T: now also XIO.16; no longer XIO.30
- net U2-E: now also XIO.14; no longer XIO.4
- net U2-T: now also XIO.11; no longer XIO.29
- net U3-E: now also XIO.18; no longer XIO.5
- net U3-T: now also XIO.15; no longer XIO.28
- net U4-E: now also XIO.17; no longer XIO.6
- net U4-T: now also XIO.20; no longer XIO.22
- net U5-E: now also XIO.6; no longer XIO.7
- net U5-T: now also XIO.5; no longer XIO.21
- net U6-E: now also XIO.7; no longer XIO.8
- net U6-T: now also XIO.8; no longer XIO.20
- net U7-E: now also XIO.21; no longer XIO.9
- net U7-T: now also XIO.22; no longer XIO.24
- net U8-E: now also XIO.24; no longer XIO.10
Routing:
- net L4: track 2.54 -> 108.5 mm, vias 0 -> 2
- net U1-E: track 0.00 -> 68.8 mm
- net U3-E: track 0.00 -> 67.7 mm
- net U4-T: track 0.00 -> 65.9 mm
- net U4-E: track 0.00 -> 65.5 mm
- net U2-E: track 0.00 -> 65.4 mm
- net L3: track 2.54 -> 61.7 mm, vias 0 -> 2
- net U2-T: track 113.4 -> 60.0 mm
- net SDA: track 2.54 -> 54.7 mm
- net RESET: track 9.04 -> 59.5 mm
- net SCL: track 2.54 -> 51.7 mm
- net IR2: track 0.00 -> 47.5 mm
- net IR4: track 0.00 -> 47.4 mm
- net L9: track 4.76 -> 50.5 mm
- net IR1: track 0.00 -> 43.3 mm
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- removed copper zone on layer 16, net N$2
Other:
- board size 93.4 x 53.3 mm -> 94.2 x 53.3 mm
- board text added: "# = PWM Pin Used by Shield"
- board text added: "Arduino Mega R3 Robot IO Shield"
- board text added: "RST"
- board text added: "version 20170223"
- board text removed: "# = Used by Shield"
- board text removed: "L5"
- board text removed: "L6"
- board text removed: "L7"
- board text removed: "L8"
- board text removed: "L9"
- board text removed: "RESET"
