File: Arduino_MEGA_2560-Rev3_Shield.sch (EAGLE design)
At the start: 44 parts, among them IC1 785.0RECOM

Commit message: Synching real boards with git repo
Parts:
- C1: value (none) -> 10uF
Connections:
- net N$1 renamed PB7
- net N$10 renamed SDA&2
- net N$11 renamed SCL&2
- net N$13 renamed PG5
- net N$16 renamed TX0
- net N$17 renamed RX0
- net N$19 renamed ADC7
- net N$20 renamed ADC6
- net N$21 renamed ADC5
- net N$22 renamed ADC4
- net N$23 renamed ADC3
- net N$24 renamed ADC2
- net N$25 renamed ADC1
- net N$26 renamed ADC0
- net N$3 renamed PB6
- net N$4 renamed PB5
- net N$5 renamed PB4
- net N$8 renamed TXD1
- net N$9 renamed RXD1
- removed net N$6: JP1.9, JP6.9
- removed net PD7: XIO.19
- new net PC6: XIO.12
- new net PE3: PWML.6, PWML1.6
- net IR1: now also XIO.3; no longer XIO.18
- net IR2: now also XIO.4; no longer XIO.17
- net IR3: now also XIO.19; no longer XIO.16
- net IR4: now also XIO.28; no longer XIO.15
- net IR5: now also XIO.9; no longer XIO.14
- net IR6: now also XIO.10; no longer XIO.13
- net IR7: now also XIO.29; no longer XIO.12
- net IR8: now also XIO.30; no longer XIO.11
- net L1: now also PWML.8, PWML1.8; no longer PWML.6, PWML1.6
- net L2: now also PWML.7, PWML1.7; no longer PWML.3, PWML1.3
- net L3: now also JP1.10, JP6.10; no longer PWML.4, PWML1.4
- net L4: now also JP1.9, JP6.9; no longer PWML.7, PWML1.7
- net L5: now also XIO.27; no longer PWML.8, PWML1.8
- net L6: now also XIO.26; no longer JP1.10, JP6.10
- net L7: now also XIO.25; no longer XIO.27
- net L8: now also PWML.3, PWML1.3; no longer XIO.26
- net L9: now also PWML.4, PWML1.4; no longer XIO.25
- net U1-E: now also XIO.13; no longer XIO.3
- net U1-T: now also XIO.16; no longer XIO.30
- net U2-E: now also XIO.14; no longer XIO.4
- net U2-T: now also XIO.11; no longer XIO.29
- net U3-E: now also XIO.18; no longer XIO.5
- net U3-T: now also XIO.15; no longer XIO.28
- net U4-E: now also XIO.17; no longer XIO.6
- net U4-T: now also XIO.20; no longer XIO.22
- net U5-E: now also XIO.6; no longer XIO.7
- net U5-T: now also XIO.5; no longer XIO.21
- net U6-E: now also XIO.7; no longer XIO.8
- net U6-T: now also XIO.8; no longer XIO.20
- net U7-E: now also XIO.21; no longer XIO.9
- net U7-T: now also XIO.22; no longer XIO.24
- net U8-E: now also XIO.24; no longer XIO.10
Other:
- note added: "OC0A/OC1C"
- note added: "OC0B"
- note added: "OC1A"
- note added: "OC1B"
- note added: "OC2A"
- note added: "OC2B"
- note added: "OC3A"
- note added: "OC3B"
- note added: "OC3C"
- note added: "OC4A"
- note added: "OC4B"
- note added: "OC4C"
- note added: "OC5A"
- note added: "OC5B"
- note added: "OC5C"
- note added: "PA0"
- note added: "PA1"
- note added: "PA2"
- note added: "PA3"
- note added: "PA4"
- note added: "PA5"
- note added: "PA6"
- note added: "PA7"
- note added: "PB0"
- note added: "PB1"
- note added: "PB2"
- note added: "PB3"
- note added: "PB4"
- note added: "PB5"
- note added: "PB6"
- note added: "PB7"
- note added: "PC0"
- note added: "PC1"
- note added: "PC2"
- note added: "PC3"
- note added: "PC4"
- note added: "PC5"
- note added: "PC6"
- note added: "PC7"
- note added: "PD7"
- note added: "PE0"
- note added: "PE1"
- note added: "PE3"
- note added: "PE4"
- note added: "PE5"
- note added: "PG0"
- note added: "PG1"
- note added: "PG2"
- note added: "PG5"
- note added: "PH3"
- note added: "PH4"
- note added: "PH5"
- note added: "PH6"
- note added: "PL0"
- note added: "PL1"
- note added: "PL2"
- note added: "PL3"
- note added: "PL4"
- note added: "PL5"
- note added: "PL6"
- note added: "PL7"
- note added: "PWM"
- note added: "SCL"
- note added: "SDA"
- moved on the sheet: IR1, IR2, IR3, IR4, IR5, IR6, IR7, IR8, L1, L2, L3, L4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
